File: stemthortyto.kicad_sch (KiCad schematic)
At the start: 17 parts, among them IC1 E22-900M22S, J1 UART Connectors, J2 I2C Connectors, J3 5022442430, U1 STM32H743VITx, U2 ADXL343

Commit message: Add files via upload
Parts:
- removed C4: 0.1μF, symbol Device:C_Small
- removed J1: UART Connectors, symbol Connector:Conn_01x05_Pin
- removed J2: I2C Connectors, symbol Connector:Conn_01x02_Pin
- removed J3: 5022442430, 5022442430:CONN_502244-2430_MOL, symbol 5022442430:5022442430
- removed R3, R4, R5, R6: 220, symbol Device:R
- removed U1: STM32H743VITx, Package_QFP:LQFP-100_14x14mm_P0.5mm, symbol MCU_ST_STM32H7:STM32H743VITx
- added C10, C11, C12, C13, C14, C16, C17, C18, C19, C20, C21, C22, C23, C24, C25, C27, C28, C29, C30, C31, C32, C5, C6, C7, C8, C9: 0.1μf, Capacitor_SMD:C_0201_0603Metric, symbol Device:C_Small
- added C15, C26, C39: 4.7μf, Capacitor_SMD:C_01005_0402Metric, symbol Device:C_Small
- added C33: 1μf, symbol Device:C_Small
- added C34: 10pF, symbol Device:C_Small
- added C35, C37, C40: 0.1μF, symbol Device:C_Small
- added C36, C38: 4.7μF, symbol Device:C_Small
- added D1: LED, symbol Device:LED
- added Q1: BCV29, Package_TO_SOT_SMD:SOT-89-3, symbol Transistor_BJT:BCV29
- added R10: 4.7k, Resistor_SMD:R_0402_1005Metric, symbol Device:R_Small
- added R11, R12, R9: 10K, Resistor_SMD:R_0402_1005Metric, symbol Device:R_Small
- added R13: R_Small, Resistor_SMD:R_0402_1005Metric, symbol Device:R_Small
- added R14: 0, Resistor_SMD:R_0402_1005Metric, symbol Device:R_Small
- added R3: 4.7K, symbol Device:R_Small
- added R4: 48, symbol Device:R_Small
- added R5, R6: 200, symbol Device:R_Small
- added R7, R8: 240, Resistor_SMD:R_0402_1005Metric, symbol Device:R_Small
- added U3: RK3588S, symbol RK3588S:RK3588S
- added U4: K4UCE3Q4AB-MGCL, easyeda2kicad:FBGA-200_L15.0-W10.0-BL_RS512M32LO4D1BDS-53BT, symbol easyeda2kicad:K4UCE3Q4AB-MGCL
- added U5: FEMDRW032G-88A19, easyeda2kicad:FBGA-153_L13.0-W11.5-P0.50_KLMAG1JETD-B041, symbol friggineda:FEMDRW032G-88A19
- C1, C2, C3: footprint (none) -> Capacitor_SMD:C_0201_0603Metric
- R1, R2: value 4.7K -> 2.7K; footprint (none) -> Resistor_SMD:R_0402_1005Metric
Connections:
- net +3.3V: now also C36.1, C37.1, R3.1, R4.1, U5.E6 (VCC), U5.F5 (VCC), U5.J10 (VCC), U5.K9 (VCC)
- net GND: now also C10.2, C11.2, C12.2, C13.2, C14.2, C15.2, C16.2, C17.2, C18.2, C19.2, C20.2, C21.2, C22.2, C23.2, C24.2, C25.2, C26.2, C27.2, C28.2, C29.2, C30.2, C31.2, C32.2, C33.1, C34.2, C35.2, C36.2, C37.2, C38.2, C39.2, C40.2, C5.2, C6.2, C7.2, C8.2, C9.2, Q1.3 (E), R10.2, U4.A10 (VSS), U4.A3 (VSS), U4.AB10 (VSS), U4.AB3 (VSS), U4.AB5 (VSS), U4.AB8 (VSS), U4.C1 (VSS), U4.C12 (VSS), U4.C5 (VSS), U4.C8 (VSS), U4.D11 (VSS), U4.D2 (VSS), U4.D4 (VSS), U4.D9 (VSS), U4.E1 (VSS), U4.E12 (VSS), U4.E5 (VSS), U4.E8 (VSS), U4.G1 (VSS), U4.G10 (VSS), U4.G12 (VSS), U4.G3 (VSS), U4.G5 (VSS), U4.G8 (VSS), U4.J1 (VSS), U4.J10 (VSS), U4.J12 (VSS), U4.J3 (VSS), U4.K11 (VSS), U4.K2 (VSS), U4.K4 (VSS), U4.K9 (VSS), U4.N11 (VSS), U4.N2 (VSS), U4.N4 (VSS), U4.N9 (VSS), U4.P1 (VSS), U4.P10 (VSS), U4.P12 (VSS), U4.P3 (VSS), U4.T1 (VSS), U4.T10 (VSS), U4.T12 (VSS), U4.T3 (VSS), U4.T5 (VSS), U4.T8 (VSS), U4.V1 (VSS), U4.V12 (VSS), U4.V5 (VSS), U4.V8 (VSS), U4.W11 (VSS), U4.W2 (VSS), U4.W4 (VSS), U4.W9 (VSS), U4.Y1 (VSS), U4.Y12 (VSS), U4.Y5 (VSS), U4.Y8 (VSS), U5.C4 (VSSQ), U5.E7 (VSS), U5.G5 (VSS), U5.H10 (VSS), U5.J5 (VSS), U5.K8 (VSS), U5.N2 (VSSQ), U5.N5 (VSSQ), U5.P4 (VSSQ), U5.P6 (VSSQ)
- net LoRaBUSY: now reaches IC1.14 (BUSY)
- net LoRaBUSY: now also Q1.1 (B)
- net LoRaRST: now reaches IC1.15 (NRST)
- net LoRaRST: now also R3.2, U3.H38 (PDM1_SDI0_M1/PCIE20X1_1_PERSTN_M2/PWM3_IR_M3/SPI2_CS0_M0/GPIO1_A7_u)
- net LoRaMISO: now reaches IC1.16 (MISO)
- net LoRaMISO: now also U3.AV19 (CIF_D0/BT1120_D0/I2S1_MCLK_M0/PCIE20X1_1_CLKREQN_M1/UART9_RTSN_M1/SPI0_MISO_M1/GPIO4_A0_d)
- net LoRaMOSI: now reaches IC1.17 (MOSI)
- net LoRaMOSI: now also U3.AW18 (CIF_D1/BT1120_D1/I2S1_SCLK_TX_M0/PCIE20X1_1_WAKEN_M1/UART9_CTSN_M1/SPI0_MOSI_M1/GPIO4_A1_d)
- net LoRaSCK(CK): now reaches IC1.18 (SCK)
- net LoRaSCK(CK): now also U3.AV26 (CIF_D2/BT1120_D2/I2S1_LRCK_TX_M0/PCIE20X1_1_PERSTN_M1/SPI0_CLK_M1/GPIO4_A2_d)
- net LoRaCS: now reaches IC1.19 (NSS)
- net LoRaCS: now also U3.AT15 (CIF_HREF/BT1120_D8/I2S1_SDO1_M0/PCIE20X1_1_BUTTON_RSTN/I2C7_SCL_M3/UART8_RTSN_M0/PWM14_M1/SPI0_CS0_M1/CAN1_RX_M1/GPIO4_B2_u)
- net LoRaRX: now reaches IC1.6 (RXEN)
- net LoRaRX: now also R5.1
- net LoRaTX: now reaches IC1.7 (TXEN)
- net LoRaTX: now also R6.1
- net SDAACCL: now reaches R1.2, U2.13 (SDA/SDI/SDIO)
- net SDAACCL: now also U3.AH40 (I2S1_SCLK_TX_M1/JTAG_TMS_M2/I2C1_SDA_M0/UART2_RX_M0/PCIE20X1_1_WAKEN_M0/GPIO0_B6_d), U3.AM39 (I2S1_SDO3_M1/CPU_BIG1_AVS/I2C1_SDA_M2/CAN2_TX_M1/HDMI_TX0_SCL_M1/SPI3_CS1_M2/SATA_MP_SWITCH/GPIO0_D5_u)
- net SCLACCL: now reaches R2.2, U2.14 (SCL/SCLK)
- net SCLACCL: now also U3.AH39 (I2S1_MCLK_M1/JTAG_TCK_M2/I2C1_SCL_M0/UART2_TX_M0/PCIE20X1_1_CLKREQN_M0/GPIO0_B5_d), U3.AL39 (I2S1_SDO2_M1/PDM0_SDI2_M1/PWM3_IR_M0/I2C1_SCL_M2/CAN2_RX_M1/HDMI_TX0_SDA_M1/SPI3_CS0_M2/SATA_CPDET/GPIO0_D4_u)
- new net: R5.2, U3.G40 (PCIE20X1_1_CLKREQN_M2/DP0_HPDIN_M2/I2C2_SDA_M4/UART6_RX_M1/SPI4_MISO_M2/GPIO1_A0_d)
- new net: C34.1, R13.2, U5.M6 (CLK)
- new net: R7.2, U4.A5 (ZQ0)
- new net: R8.2, U4.A8 (ZQ1)
- new net: R10.1, U4.G2 (ODT_CA_a1)/2)), U4.T2 (ODT_CA_b1)/2))
- new net: U3.A1 (VSS[533]), U3.A2 (VSS[533]), U3.A42 (VSS[533]), U3.AA10 (VSS[533]), U3.AA11 (VSS[533]), U3.AA12 (VSS[533]), U3.AA19 (VSS[533]), U3.AA22 (VSS[533]), U3.AA23 (VSS[533]), U3.AA3 (VSS[533]), U3.AA31 (VSS[533]), U3.AA37 (VSS[533]), U3.AA38 (VSS[533]), U3.AA39 (VSS[533]), U3.AA40 (VSS[533]), U3.AA6 (VSS[533]), U3.AA7 (VSS[533]), U3.AA8 (VSS[533]), U3.AA9 (VSS[533]), U3.AB10 (VSS[533]), U3.AB11 (VSS[533]), U3.AB12 (VSS[533]), U3.AB19 (VSS[533]), U3.AB2 (VSS[533]), U3.AB20 (VSS[533]), U3.AB21 (VSS[533]), U3.AB22 (VSS[533]), U3.AB23 (VSS[533]), U3.AB24 (VSS[533]), U3.AB32 (VSS[533]), U3.AB33 (VSS[533]), U3.AB34 (VSS[533]), U3.AB36 (VSS[533]), U3.AB37 (VSS[533]), U3.AB38 (VSS[533]), U3.AB39 (VSS[533]), U3.AB40 (VSS[533]), U3.AB6 (VSS[533]), U3.AB9 (VSS[533]), U3.AC17 (VSS[533]), U3.AC18 (VSS[533]), U3.AC22 (VSS[533]), U3.AC23 (VSS[533]), U3.AC24 (VSS[533]), U3.AC25 (VSS[533]), U3.AC26 (VSS[533]), U3.AC3 (VSS[533]), U3.AC4 (VSS[533]), U3.AC41 (VSS[533]), U3.AC5 (VSS[533]), U3.AC6 (VSS[533]), U3.AD10 (VSS[533]), U3.AD11 (VSS[533]), U3.AD12 (VSS[533]), U3.AD13 (VSS[533]), U3.AD14 (VSS[533]), U3.AD19 (VSS[533]), U3.AD2 (VSS[533]), U3.AD20 (VSS[533]), U3.AD22 (VSS[533]), U3.AD23 (VSS[533]), U3.AD24 (VSS[533]), U3.AD25 (VSS[533]), U3.AD3 (VSS[533]), U3.AD5 (VSS[533]), U3.AD6 (VSS[533]), U3.AD8 (VSS[533]), U3.AD9 (VSS[533]), U3.AE10 (VSS[533]), U3.AE11 (VSS[533]), U3.AE12 (VSS[533]), U3.AE13 (VSS[533]), U3.AE14 (VSS[533]), U3.AE15 (VSS[533]), U3.AE16 (VSS[533]), U3.AE19 (VSS[533]), U3.AE20 (VSS[533]), U3.AE22 (VSS[533]), U3.AE23 (VSS[533]), U3.AE24 (VSS[533]), U3.AE25 (VSS[533]), U3.AE26 (VSS[533]), U3.AE38 (VSS[533]), U3.AE39 (VSS[533]), U3.AE40 (VSS[533]), U3.AE6 (VSS[533]), U3.AE7 (VSS[533]), U3.AE8 (VSS[533]), U3.AE9 (VSS[533]), U3.AF10 (VSS[533]), U3.AF16 (VSS[533]), U3.AF17 (VSS[533]), U3.AF19 (VSS[533]), U3.AF2 (VSS[533]), U3.AF20 (VSS[533]), U3.AF21 (VSS[533]), U3.AF26 (VSS[533]), U3.AF27 (VSS[533]), U3.AF28 (VSS[533]), U3.AF29 (VSS[533]), U3.AF30 (VSS[533]), U3.AF31 (VSS[533]), U3.AF32 (VSS[533]), U3.AF33 (VSS[533]), U3.AF34 (VSS[533]), U3.AF37 (VSS[533]), U3.AF38 (VSS[533]), U3.AF39 (VSS[533]), U3.AF40 (VSS[533]), U3.AF41 (VSS[533]), U3.AF6 (VSS[533]), U3.AF7 (VSS[533]), U3.AF8 (VSS[533]), U3.AF9 (VSS[533]), U3.AG15 (VSS[533]), U3.AG16 (VSS[533]), U3.AG17 (VSS[533]), U3.AG18 (VSS[533]), U3.AG19 (VSS[533]), U3.AG20 (VSS[533]), U3.AG21 (VSS[533]), U3.AG22 (VSS[533]), U3.AG23 (VSS[533]), U3.AG24 (VSS[533]), U3.AG25 (VSS[533]), U3.AG28 (VSS[533]), U3.AG29 (VSS[533]), U3.AG3 (VSS[533]), U3.AG31 (VSS[533]), U3.AG32 (VSS[533]), U3.AG33 (VSS[533]), U3.AG34 (VSS[533]), U3.AG35 (VSS[533]), U3.AG4 (VSS[533]), U3.AG40 (VSS[533]), U3.AG5 (VSS[533]), U3.AG6 (VSS[533]), U3.AG7 (VSS[533]), U3.AG8 (VSS[533]), U3.AH10 (VSS[533]), U3.AH16 (VSS[533]), U3.AH17 (VSS[533]), U3.AH2 (VSS[533]), U3.AH28 (VSS[533]), U3.AH29 (VSS[533]), U3.AH3 (VSS[533]), U3.AH36 (VSS[533]), U3.AH4 (VSS[533]), U3.AH5 (VSS[533]), U3.AH7 (VSS[533]), U3.AH8 (VSS[533]), U3.AH9 (VSS[533]), U3.AJ10 (VSS[533]), U3.AJ11 (VSS[533]), U3.AJ12 (VSS[533]), U3.AJ16 (VSS[533]), U3.AJ26 (VSS[533]), U3.AJ27 (VSS[533]), U3.AJ28 (VSS[533]), U3.AJ29 (VSS[533]), U3.AJ30 (VSS[533]), U3.AJ35 (VSS[533]), U3.AJ38 (VSS[533]), U3.AJ39 (VSS[533]), U3.AJ40 (VSS[533]), U3.AJ41 (VSS[533]), U3.AJ5 (VSS[533]), U3.AJ7 (VSS[533]), U3.AJ8 (VSS[533]), U3.AJ9 (VSS[533]), U3.AK16 (VSS[533]), U3.AK2 (VSS[533]), U3.AK22 (VSS[533]), U3.AK26 (VSS[533]), U3.AK30 (VSS[533]), U3.AK40 (VSS[533]), U3.AK6 (VSS[533]), U3.AK7 (VSS[533]), U3.AL16 (VSS[533]), U3.AL22 (VSS[533]), U3.AL3 (VSS[533]), U3.AL35 (VSS[533]), U3.AL4 (VSS[533]), U3.AL5 (VSS[533]), U3.AM16 (VSS[533]), U3.AM17 (VSS[533]), U3.AM23 (VSS[533]), U3.AM25 (VSS[533]), U3.AM27 (VSS[533]), U3.AM31 (VSS[533]), U3.AM32 (VSS[533]), U3.AM4 (VSS[533]), U3.AM41 (VSS[533]), U3.AM5 (VSS[533]), U3.AN17 (VSS[533]), U3.AN23 (VSS[533]), U3.AN25 (VSS[533]), U3.AN3 (VSS[533]), U3.AN31 (VSS[533]), U3.AN32 (VSS[533]), U3.AN33 (VSS[533]), U3.AN34 (VSS[533]), U3.AN35 (VSS[533]), U3.AN37 (VSS[533]), U3.AN38 (VSS[533]), U3.AN39 (VSS[533]), U3.AN40 (VSS[533]), U3.AN6 (VSS[533]), U3.AN7 (VSS[533]), U3.AP2 (VSS[533]), U3.AP25 (VSS[533]), U3.AP27 (VSS[533]), U3.AP33 (VSS[533]), U3.AP34 (VSS[533]), U3.AP35 (VSS[533]), U3.AP37 (VSS[533]), U3.AP38 (VSS[533]), U3.AP39 (VSS[533]), U3.AP40 (VSS[533]), U3.AP5 (VSS[533]), U3.AP6 (VSS[533]), U3.AR3 (VSS[533]), U3.AR4 (VSS[533]), U3.AR40 (VSS[533]), U3.AR41 (VSS[533]), U3.AT2 (VSS[533]), U3.AT36 (VSS[533]), U3.AT5 (VSS[533]), U3.AT6 (VSS[533]), U3.AU2 (VSS[533]), U3.AU3 (VSS[533]), U3.AU35 (VSS[533]), U3.AU38 (VSS[533]), U3.AU39 (VSS[533]), U3.AU4 (VSS[533]), U3.AU40 (VSS[533]), U3.AV36 (VSS[533]), U3.AV41 (VSS[533]), U3.AV5 (VSS[533]), U3.AW3 (VSS[533]), U3.AW4 (VSS[533]), U3.B10 (VSS[533]), U3.B11 (VSS[533]), U3.B14 (VSS[533]), U3.B17 (VSS[533]), U3.B19 (VSS[533]), U3.B21 (VSS[533]), U3.B23 (VSS[533]), U3.B26 (VSS[533]), U3.B27 (VSS[533]), U3.B29 (VSS[533]), U3.B3 (VSS[533]), U3.B31 (VSS[533]), U3.B34 (VSS[533]), U3.B35 (VSS[533]), U3.B36 (VSS[533]), U3.B38 (VSS[533]), U3.B40 (VSS[533]), U3.B42 (VSS[533]), U3.B5 (VSS[533]), U3.B8 (VSS[533]), U3.C11 (VSS[533]), U3.C12 (VSS[533]), U3.C14 (VSS[533]), U3.C15 (VSS[533]), U3.C18 (VSS[533]), U3.C19 (VSS[533]), U3.C2 (VSS[533]), U3.C20 (VSS[533]), U3.C22 (VSS[533]), U3.C24 (VSS[533]), U3.C26 (VSS[533]), U3.C28 (VSS[533]), U3.C30 (VSS[533]), U3.C35 (VSS[533]), U3.C37 (VSS[533]), U3.C39 (VSS[533]), U3.C6 (VSS[533]), U3.C7 (VSS[533]), U3.C9 (VSS[533]), U3.D11 (VSS[533]), U3.D14 (VSS[533]), U3.D15 (VSS[533]), U3.D18 (VSS[533]), U3.D19 (VSS[533]), U3.D22 (VSS[533]), U3.D26 (VSS[533]), U3.D3 (VSS[533]), U3.D30 (VSS[533]), U3.D31 (VSS[533]), U3.D32 (VSS[533]), U3.D4 (VSS[533]), U3.D7 (VSS[533]), U3.E10 (VSS[533]), U3.E12 (VSS[533]), U3.E16 (VSS[533]), U3.E18 (VSS[533]), U3.E19 (VSS[533]), U3.E2 (VSS[533]), U3.E21 (VSS[533]), U3.E23 (VSS[533]), U3.E25 (VSS[533]), U3.E27 (VSS[533]), U3.E30 (VSS[533]), U3.E31 (VSS[533]), U3.E33 (VSS[533]), U3.E34 (VSS[533]), U3.E37 (VSS[533]), U3.E38 (VSS[533]), U3.E39 (VSS[533]), U3.E5 (VSS[533]), U3.E6 (VSS[533]), U3.E8 (VSS[533]), U3.E9 (VSS[533]), U3.F10 (VSS[533]), U3.F13 (VSS[533]), U3.F14 (VSS[533]), U3.F15 (VSS[533]), U3.F16 (VSS[533]), U3.F19 (VSS[533]), U3.F2 (VSS[533]), U3.F21 (VSS[533]), U3.F23 (VSS[533]), U3.F29 (VSS[533]), U3.F3 (VSS[533]), U3.F31 (VSS[533]), U3.F33 (VSS[533]), U3.F34 (VSS[533]), U3.F35 (VSS[533]), U3.F36 (VSS[533]), U3.F38 (VSS[533]), U3.F39 (VSS[533]), U3.F4 (VSS[533]), U3.F8 (VSS[533]), U3.F9 (VSS[533]), U3.G10 (VSS[533]), U3.G12 (VSS[533]), U3.G20 (VSS[533]), U3.G21 (VSS[533]), U3.G22 (VSS[533]), U3.G25 (VSS[533]), U3.G26 (VSS[533]), U3.G29 (VSS[533]), U3.G3 (VSS[533]), U3.G6 (VSS[533]), U3.G8 (VSS[533]), U3.G9 (VSS[533]), U3.H11 (VSS[533]), U3.H12 (VSS[533]), U3.H22 (VSS[533]), U3.H25 (VSS[533]), U3.H29 (VSS[533]), U3.H3 (VSS[533]), U3.H4 (VSS[533]), U3.H5 (VSS[533]), U3.H6 (VSS[533]), U3.J10 (VSS[533]), U3.J12 (VSS[533]), U3.J14 (VSS[533]), U3.J15 (VSS[533]), U3.J16 (VSS[533]), U3.J2 (VSS[533]), U3.J22 (VSS[533]), U3.J24 (VSS[533]), U3.J26 (VSS[533]), U3.J29 (VSS[533]), U3.J30 (VSS[533]), U3.J31 (VSS[533]), U3.J6 (VSS[533]), U3.J7 (VSS[533]), U3.J8 (VSS[533]), U3.J9 (VSS[533]), U3.K10 (VSS[533]), U3.K11 (VSS[533]), U3.K12 (VSS[533]), U3.K14 (VSS[533]), U3.K17 (VSS[533]), U3.K22 (VSS[533]), U3.K23 (VSS[533]), U3.K25 (VSS[533]), U3.K26 (VSS[533]), U3.K3 (VSS[533]), U3.K31 (VSS[533]), U3.K32 (VSS[533]), U3.K33 (VSS[533]), U3.K6 (VSS[533]), U3.K7 (VSS[533]), U3.L10 (VSS[533]), U3.L11 (VSS[533]), U3.L12 (VSS[533]), U3.L14 (VSS[533]), U3.L2 (VSS[533]), U3.L22 (VSS[533]), U3.L23 (VSS[533]), U3.L24 (VSS[533]), U3.L3 (VSS[533]), U3.L32 (VSS[533]), U3.L33 (VSS[533]), U3.L36 (VSS[533]), U3.L5 (VSS[533])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
- new net: U3.AA14 (AVSS[132]), U3.AA26 (AVSS[132]), U3.AL15 (AVSS[132]), U3.AM14 (AVSS[132]), U3.AM15 (AVSS[132]), U3.AN11 (AVSS[132]), U3.AN13 (AVSS[132]), U3.AN14 (AVSS[132]), U3.AN15 (AVSS[132]), U3.AN18 (AVSS[132]), U3.AP10 (AVSS[132]), U3.AP11 (AVSS[132]), U3.AP16 (AVSS[132]), U3.AP22 (AVSS[132]), U3.AP31 (AVSS[132]), U3.AP32 (AVSS[132]), U3.AP7 (AVSS[132]), U3.AP8 (AVSS[132]), U3.AP9 (AVSS[132]), U3.AR16 (AVSS[132]), U3.AR18 (AVSS[132]), U3.AR20 (AVSS[132]), U3.AR21 (AVSS[132]), U3.AR22 (AVSS[132]), U3.AR25 (AVSS[132]), U3.AR9 (AVSS[132]), U3.AT16 (AVSS[132]), U3.AT19 (AVSS[132]), U3.AT20 (AVSS[132]), U3.AT21 (AVSS[132]), U3.AT22 (AVSS[132]), U3.AT23 (AVSS[132]), U3.AT29 (AVSS[132]), U3.AT7 (AVSS[132]), U3.AT8 (AVSS[132]), U3.AU16 (AVSS[132]), U3.AU18 (AVSS[132]), U3.AU19 (AVSS[132]), U3.AU21 (AVSS[132]), U3.AU24 (AVSS[132]), U3.AU25 (AVSS[132]), U3.AU27 (AVSS[132]), U3.AU28 (AVSS[132]), U3.AU29 (AVSS[132]), U3.AU31 (AVSS[132]), U3.AU8 (AVSS[132]), U3.AV12 (AVSS[132]), U3.AV14 (AVSS[132]), U3.AV15 (AVSS[132]), U3.AV16 (AVSS[132]), U3.AV21 (AVSS[132]), U3.AV25 (AVSS[132]), U3.AV29 (AVSS[132]), U3.AV32 (AVSS[132]), U3.AV33 (AVSS[132]), U3.AV8 (AVSS[132]), U3.AV9 (AVSS[132]), U3.AW12 (AVSS[132]), U3.AW14 (AVSS[132]), U3.AW16 (AVSS[132]), U3.AW17 (AVSS[132]), U3.AW21 (AVSS[132]), U3.AW25 (AVSS[132]), U3.AW28 (AVSS[132]), U3.AW29 (AVSS[132]), U3.AW32 (AVSS[132]), U3.AW33 (AVSS[132]), U3.AW36 (AVSS[132]), U3.AW40 (AVSS[132]), U3.AW8 (AVSS[132]), U3.AW9 (AVSS[132]), U3.AY12 (AVSS[132]), U3.AY14 (AVSS[132]), U3.AY16 (AVSS[132]), U3.AY17 (AVSS[132]), U3.AY18 (AVSS[132]), U3.AY2 (AVSS[132]), U3.AY21 (AVSS[132]), U3.AY22 (AVSS[132]), U3.AY23 (AVSS[132]), U3.AY25 (AVSS[132]), U3.AY28 (AVSS[132]), U3.AY29 (AVSS[132]), U3.AY32 (AVSS[132]), U3.AY33 (AVSS[132]), U3.AY36 (AVSS[132]), U3.AY37 (AVSS[132]), U3.AY39 (AVSS[132]), U3.AY4 (AVSS[132]), U3.AY41 (AVSS[132]), U3.AY5 (AVSS[132]), U3.AY7 (AVSS[132]), U3.AY8 (AVSS[132]), U3.AY9 (AVSS[132]), U3.BA12 (AVSS[132]), U3.BA15 (AVSS[132]), U3.BA18 (AVSS[132]), U3.BA21 (AVSS[132]), U3.BA24 (AVSS[132]), U3.BA27 (AVSS[132]), U3.BA3 (AVSS[132]), U3.BA30 (AVSS[132]), U3.BA33 (AVSS[132]), U3.BA36 (AVSS[132]), U3.BA6 (AVSS[132]), U3.BA9 (AVSS[132]), U3.BB1 (AVSS[132]), U3.BB42 (AVSS[132]), U3.C41 (AVSS[132]), U3.E40 (AVSS[132]), U3.F40 (AVSS[132]), U3.G36 (AVSS[132]), U3.G41 (AVSS[132]), U3.H37 (AVSS[132]), U3.H40 (AVSS[132]), U3.J38 (AVSS[132]), U3.J39 (AVSS[132]), U3.J40 (AVSS[132]), U3.K34 (AVSS[132]), U3.K35 (AVSS[132]), U3.K36 (AVSS[132]), U3.K37 (AVSS[132]), U3.K38 (AVSS[132]), U3.K39 (AVSS[132]), U3.K40 (AVSS[132]), U3.L34 (AVSS[132]), U3.L35 (AVSS[132]), U3.L41 (AVSS[132]), U3.M33 (AVSS[132]), U3.M34 (AVSS[132]), U3.N15 (AVSS[132]), U3.N33 (AVSS[132])
- new net: U3.AA28 (VDD_CPU_LIT[12]), U3.AA29 (VDD_CPU_LIT[12]), U3.AA30 (VDD_CPU_LIT[12]), U3.AB31 (VDD_CPU_LIT[12]), U3.AC27 (VDD_CPU_LIT[12]), U3.AC28 (VDD_CPU_LIT[12]), U3.AC29 (VDD_CPU_LIT[12]), U3.AC30 (VDD_CPU_LIT[12]), U3.AC31 (VDD_CPU_LIT[12]), U3.AD26 (VDD_CPU_LIT[12]), U3.AD27 (VDD_CPU_LIT[12]), U3.AE27 (VDD_CPU_LIT[12])
- new net: U3.AC16 (VDD_VDENC[9]), U3.AD15 (VDD_VDENC[9]), U3.P15 (VDD_VDENC[9]), U3.R15 (VDD_VDENC[9]), U3.T15 (VDD_VDENC[9]), U3.U15 (VDD_VDENC[9]), U3.W16 (VDD_VDENC[9]), U3.W17 (VDD_VDENC[9]), U3.Y17 (VDD_VDENC[9])
- new net: U3.AC33 (VCCIO5[2]), U3.AC34 (VCCIO5[2])
- new net: U3.AF12 (VDD_LOGIC[18]), U3.AF13 (VDD_LOGIC[18]), U3.AH11 (VDD_LOGIC[18]), U3.AH12 (VDD_LOGIC[18]), U3.AH13 (VDD_LOGIC[18]), U3.AH14 (VDD_LOGIC[18]), U3.AH15 (VDD_LOGIC[18]), U3.AH23 (VDD_LOGIC[18]), U3.AH24 (VDD_LOGIC[18]), U3.AJ15 (VDD_LOGIC[18]), U3.AJ31 (VDD_LOGIC[18]), U3.AJ32 (VDD_LOGIC[18]), U3.AK15 (VDD_LOGIC[18]), U3.AL31 (VDD_LOGIC[18]), U3.H27 (VDD_LOGIC[18]), U3.J27 (VDD_LOGIC[18]), U3.W33 (VDD_LOGIC[18]), U3.Y33 (VDD_LOGIC[18])
- new net: U3.AH18 (VDD_GPU[13]), U3.AH19 (VDD_GPU[13]), U3.AH20 (VDD_GPU[13]), U3.AH21 (VDD_GPU[13]), U3.AJ19 (VDD_GPU[13]), U3.AJ20 (VDD_GPU[13]), U3.AJ21 (VDD_GPU[13]), U3.AK21 (VDD_GPU[13]), U3.AL21 (VDD_GPU[13]), U3.AM21 (VDD_GPU[13]), U3.AM22 (VDD_GPU[13]), U3.AN21 (VDD_GPU[13]), U3.AN22 (VDD_GPU[13])
- new net: U3.AH25 (VDD_NPU_MEM[4]), U3.AH26 (VDD_NPU_MEM[4]), U3.AJ25 (VDD_NPU_MEM[4]), U3.AK25 (VDD_NPU_MEM[4])
- new net: U3.AJ18 (VDD_GPU_MEM[3]), U3.AK18 (VDD_GPU_MEM[3]), U3.AL18 (VDD_GPU_MEM[3])
- new net: U3.AK27 (VDD_NPU[9]), U3.AK28 (VDD_NPU[9]), U3.AK29 (VDD_NPU[9]), U3.AL28 (VDD_NPU[9]), U3.AL29 (VDD_NPU[9]), U3.AL30 (VDD_NPU[9]), U3.AM30 (VDD_NPU[9]), U3.AN30 (VDD_NPU[9]), U3.AP30 (VDD_NPU[9])
- new net: U3.AL33 (VCCIO6[2]), U3.AM33 (VCCIO6[2])
- new net: U3.AM13 (HDMI/eDP_TX0_VDD_0V75[2]), U3.AN12 (HDMI/eDP_TX0_VDD_0V75[2])
- new net: U3.AP18 (TYPEC0_DP0_VDDA_0V85[2]), U3.AR19 (TYPEC0_DP0_VDDA_0V85[2])
- new net: U3.G27 (VCCIO4_1V8[2]), U3.G28 (VCCIO4_1V8[2])
- new net: U3.H14 (DDR_CH1_VDDQ[5]), U3.H15 (DDR_CH1_VDDQ[5]), U3.H16 (DDR_CH1_VDDQ[5]), U3.H18 (DDR_CH1_VDDQ[5]), U3.H20 (DDR_CH1_VDDQ[5])
- new net: U3.J18 (DDR_CH1_VDD[3]), U3.K18 (DDR_CH1_VDD[3]), U3.L18 (DDR_CH1_VDD[3])
- new net: U3.J20 (DDR_CH1_VDD_MIF[3]), U3.K20 (DDR_CH1_VDD_MIF[3]), U3.L20 (DDR_CH1_VDD_MIF[3])
- new net: U3.K27 (VDD_CPU_BIG0[14]), U3.K28 (VDD_CPU_BIG0[14]), U3.K29 (VDD_CPU_BIG0[14]), U3.K30 (VDD_CPU_BIG0[14]), U3.M24 (VDD_CPU_BIG0[14]), U3.M25 (VDD_CPU_BIG0[14]), U3.M28 (VDD_CPU_BIG0[14]), U3.M29 (VDD_CPU_BIG0[14]), U3.M30 (VDD_CPU_BIG0[14]), U3.N24 (VDD_CPU_BIG0[14]), U3.N25 (VDD_CPU_BIG0[14]), U3.P23 (VDD_CPU_BIG0[14]), U3.R23 (VDD_CPU_BIG0[14]), U3.R24 (VDD_CPU_BIG0[14])
- new net: U3.P10 (DDR_CH0_VDDQ[6]), U3.R10 (DDR_CH0_VDDQ[6]), U3.T10 (DDR_CH0_VDDQ[6]), U3.V10 (DDR_CH0_VDDQ[6]), U3.W10 (DDR_CH0_VDDQ[6]), U3.Y10 (DDR_CH0_VDDQ[6])
- new net: U3.R26 (VDD_CPU_BIG1[14]), U3.R27 (VDD_CPU_BIG1[14]), U3.R28 (VDD_CPU_BIG1[14]), U3.R29 (VDD_CPU_BIG1[14]), U3.R30 (VDD_CPU_BIG1[14]), U3.R31 (VDD_CPU_BIG1[14]), U3.R32 (VDD_CPU_BIG1[14]), U3.R33 (VDD_CPU_BIG1[14]), U3.T26 (VDD_CPU_BIG1[14]), U3.U26 (VDD_CPU_BIG1[14]), U3.V26 (VDD_CPU_BIG1[14]), U3.V27 (VDD_CPU_BIG1[14]), U3.V28 (VDD_CPU_BIG1[14]), U3.V29 (VDD_CPU_BIG1[14])
- new net: U3.T12 (DDR_CH0_VDD[4]), U3.T13 (DDR_CH0_VDD[4]), U3.U12 (DDR_CH0_VDD[4]), U3.U13 (DDR_CH0_VDD[4])
- new net: U3.V12 (DDR_CH0_VDD_MIF[3]), U3.V13 (DDR_CH0_VDD_MIF[3]), U3.V14 (DDR_CH0_VDD_MIF[3])
- new net: R6.2, U3.L40 (PCIE20X1_1_WAKEN_M2/I2C2_SCL_M4/UART6_TX_M1/SPI4_MOSI_M2/GPIO1_A1_d)
- new net: D1.1 (K), Q1.2 (C)
- new net: D1.2 (A), R4.2
- new net: R14.1, U5.H5 (DS)
- new net: C33.2, U5.C2 (VDDI)
- new net: C35.1, U5.K5 (RSTN)
- new net +0V6: C10.1, C11.1, C12.1, C13.1, C14.1, C15.1, C5.1, C6.1, C7.1, C8.1, C9.1, R7.1, R8.1, U4.AA10 (VDDQ), U4.AA3 (VDDQ), U4.AA5 (VDDQ), U4.AA8 (VDDQ), U4.B10 (VDDQ), U4.B3 (VDDQ), U4.B5 (VDDQ), U4.B8 (VDDQ), U4.D1 (VDDQ), U4.D12 (VDDQ), U4.D5 (VDDQ), U4.D8 (VDDQ), U4.F10 (VDDQ), U4.F3 (VDDQ), U4.U10 (VDDQ), U4.U3 (VDDQ), U4.W1 (VDDQ), U4.W12 (VDDQ), U4.W5 (VDDQ), U4.W8 (VDDQ)
- new net +1V1: C16.1, C17.1, C18.1, C19.1, C20.1, C21.1, C22.1, C23.1, C24.1, C25.1, C26.1, C27.1, C28.1, U4.A4 (VDD2), U4.A9 (VDD2), U4.AB4 (VDD2), U4.AB9 (VDD2), U4.F5 (VDD2), U4.F8 (VDD2), U4.H1 (VDD2), U4.H12 (VDD2), U4.H5 (VDD2), U4.H8 (VDD2), U4.K1 (VDD2), U4.K10 (VDD2), U4.K12 (VDD2), U4.K3 (VDD2), U4.N1 (VDD2), U4.N10 (VDD2), U4.N12 (VDD2), U4.N3 (VDD2), U4.R1 (VDD2), U4.R12 (VDD2), U4.R5 (VDD2), U4.R8 (VDD2), U4.U5 (VDD2), U4.U8 (VDD2)
- new net +1V8: C29.1, C30.1, C31.1, C32.1, C39.1, U4.F1 (VDD1), U4.F12 (VDD1), U4.G4 (VDD1), U4.G9 (VDD1), U4.T4 (VDD1), U4.T9 (VDD1), U4.U1 (VDD1), U4.U12 (VDD1)
- new net A0A: U3.U1 (DDR_CH0_A0_A), U4.H2 (CA0_a)
- new net A0B: U3.U2 (DDR_CH0_A0_B), U4.R2 (CA0_b)
- new net A1A: U3.AC2 (DDR_CH0_A1_A), U4.J2 (CA1_a)
- new net A1B: U3.R2 (DDR_CH0_A1_B), U4.P2 (CA1_b)
- new net A2A: U3.AF1 (DDR_CH0_A2_A), U4.H9 (CA2_a)
- new net A2B: U3.R1 (DDR_CH0_A2_B), U4.R9 (CA2_b)
- new net A3A: U3.AL2 (DDR_CH0_A3_A), U4.H10 (CA3_a)
- new net A3B: U3.D2 (DDR_CH0_A3_B), U4.R10 (CA3_b)
- new net A4A: U3.Y1 (DDR_CH0_A4_A), U4.H11 (CA4_a)
- new net A4B: U3.E1 (DDR_CH0_A4_B), U4.R11 (CA4_b)
- new net A5A: U3.AG2 (DDR_CH0_A5_A), U4.J11 (CA5_a)
- new net A5B: U3.L1 (DDR_CH0_A5_B), U4.P11 (CA5_b)
- new net A6A: U3.AM2 (DDR_CH0_A6_A)
- new net A6B: U3.H1 (DDR_CH0_A6_B)
- new net CKA: U3.AA2 (DDR_CH0_CK_A), U4.J8 (CK_t_a)
- new net CKB: U3.V2 (DDR_CH0_CK_B), U4.P8 (CK_t_b)
- new net CKBA: U3.AA1 (DDR_CH0_CKB_A), U4.J9 (CK_c_a)
- new net CKBB: U3.V1 (DDR_CH0_CKB_B), U4.P9 (CK_c_b)
- new net CKE0A: U3.AK1 (DDR_CH0_LP4/4X_CKE0/LP5_CS0_A), U4.J4 (CKE0_a)
- new net CKE0B: U3.H2 (DDR_CH0_LP4/4X_CKE0/LP5_CS0_B), U4.P4 (CKE0_b)
- new net CKE1A: U3.AD1 (DDR_CH0_LP4/4X_CKE1/LP5_CS1_A), U4.J5 (CKE1_a)
- new net CKE1B: U3.F1 (DDR_CH0_LP4/4X_CKE1/LP5_CS1_B), U4.P5 (CKE1_b)
- new net CLKOUT: R13.1, U3.AB41 (EMMC_CLKOUT/GPIO2_A1_d)
- new net CMD: R11.2, U3.AE42 (EMMC_CMD/FSPI_CLK_M0/GPIO2_A0_u), U5.M5 (CMD)
- new net CS0A: U3.Y2 (DDR_CH0_LP4/4X_CS0_A), U4.H4 (CS0_a)
- new net CS0B: U3.J1 (DDR_CH0_LP4/4X_CS0_B), U4.R4 (CS0_b)
- new net CS1A: U3.AC1 (DDR_CH0_LP4/4X_CS1_A), U4.H3 (CS1_a)
- new net CS1B: U3.M1 (DDR_CH0_LP4/4X_CS1_B), U4.R3 (CS1_b)
- new net DAT0: R12.2, U3.Y41 (EMMC_D0/FSPI_D0_M0/GPIO2_D0_u), U5.A3 (DAT0)
- new net DAT1: U3.Y40 (EMMC_D1/FSPI_D1_M0/GPIO2_D1_u), U5.A4 (DAT1)
- new net DAT2: U3.AA41 (EMMC_D2/FSPI_D2_M0/GPIO2_D2_u), U5.A5 (DAT2)
- new net DAT3: U3.AA42 (EMMC_D3/FSPI_D3_M0/GPIO2_D3_u), U5.B2 (DAT3)
- new net DAT4: U3.AB42 (EMMC_D4/I2C1_SCL_M3/UART5_RX_M2/GPIO2_D4_u), U5.B3 (DAT4)
- new net DAT5: U3.AD42 (EMMC_D5/I2C1_SDA_M3/UART5_TX_M2/GPIO2_D5_u), U5.B4 (DAT5)
- new net DAT6: U3.AD41 (EMMC_D6/FSPI_CS0N_M0/GPIO2_D6_u), U5.B5 (DAT6)
- new net DAT7: U3.AE41 (EMMC_D7/FSPI_CS1N_M0/GPIO2_D7_u), U5.B6 (DAT7)
- new net DATASTROBE: R14.2, U3.AC40 (EMMC_DATA_STROBE/I2C2_SDA_M2/UART5_CTSN_M1/GPIO2_A2_d)
- new net DM0A: U3.AE1 (DDR_CH0_DM0_A), U4.C3 (DMI0_a)
- new net DM0B: U3.V5 (DDR_CH0_DM0_B), U4.Y3 (DMI0_b)
- new net DM1A: U3.AK4 (DDR_CH0_DM1_A), U4.C10 (DMI1_a)
- new net DM1B: U3.G2 (DDR_CH0_DM1_B), U4.Y10 (DMI1_b)
- new net DQ0A: U3.AJ2 (DDR_CH0_DQ0_A), U4.B2 (DQ0_a)
- new net DQ0B: U3.U3 (DDR_CH0_DQ0_B), U4.AA2 (DQ0_b)
- new net DQ10A: U3.AN4 (DDR_CH0_DQ10_A), U4.E11 (DQ10_a)
- new net DQ10B: U3.G4 (DDR_CH0_DQ10_B), U4.V11 (DQ10_b)
- new net DQ11A: U3.AJ6 (DDR_CH0_DQ11_A), U4.F11 (DQ11_a)
- new net DQ11B: U3.J4 (DDR_CH0_DQ11_B), U4.U11 (DQ11_b)
- new net DQ12A: U3.AJ3 (DDR_CH0_DQ12_A), U4.F9 (DQ12_a)
- new net DQ12B: U3.N5 (DDR_CH0_DQ12_B), U4.U9 (DQ12_b)
- new net DQ13A: U3.AK3 (DDR_CH0_DQ13_A), U4.E9 (DQ13_a)
- new net DQ13B: U3.N2 (DDR_CH0_DQ13_B), U4.V9 (DQ13_b)
- new net DQ14A: U3.AF4 (DDR_CH0_DQ14_A), U4.C9 (DQ14_a)
- new net DQ14B: U3.J5 (DDR_CH0_DQ14_B), U4.Y9 (DQ14_b)
- new net DQ15A: U3.AF5 (DDR_CH0_DQ15_A), U4.B9 (DQ15_a)
- new net DQ15B: U3.N6 (DDR_CH0_DQ15_B), U4.AA9 (DQ15_b)
- new net DQ1A: U3.AB4 (DDR_CH0_DQ1_A), U4.C2 (DQ1_a)
- new net DQ1B: U3.AA5 (DDR_CH0_DQ1_B), U4.Y2 (DQ1_b)
- new net DQ2A: U3.AJ1 (DDR_CH0_DQ2_A), U4.E2 (DQ2_a)
- new net DQ2B: U3.N1 (DDR_CH0_DQ2_B), U4.V2 (DQ2_b)
- new net DQ3A: U3.AB3 (DDR_CH0_DQ3_A), U4.F2 (DQ3_a)
- new net DQ3B: U3.U5 (DDR_CH0_DQ3_B), U4.U2 (DQ3_b)
- new net DQ4A: U3.AB5 (DDR_CH0_DQ4_A), U4.F4 (DQ4_a)
- new net DQ4B: U3.P4 (DDR_CH0_DQ4_B), U4.U4 (DQ4_b)
- new net DQ5A: U3.AE5 (DDR_CH0_DQ5_A), U4.E4 (DQ5_a)
- new net DQ5B: U3.P3 (DDR_CH0_DQ5_B), U4.V4 (DQ5_b)
- new net DQ6A: U3.AE2 (DDR_CH0_DQ6_A), U4.C4 (DQ6_a)
- new net DQ6B: U3.U4 (DDR_CH0_DQ6_B), U4.Y4 (DQ6_b)
- new net DQ7A: U3.AF3 (DDR_CH0_DQ7_A), U4.B4 (DQ7_a)
- new net DQ7B: U3.P5 (DDR_CH0_DQ7_B), U4.AA4 (DQ7_b)
- new net DQ8A: U3.AK5 (DDR_CH0_DQ8_A), U4.B11 (DQ8_a)
- new net DQ8B: U3.G5 (DDR_CH0_DQ8_B), U4.AA11 (DQ8_b)
- new net DQ9A: U3.AN5 (DDR_CH0_DQ9_A), U4.C11 (DQ9_a)
- new net DQ9B: U3.J3 (DDR_CH0_DQ9_B), U4.Y11 (DQ9_b)
- new net DQS0NA: U3.AN2 (DDR_CH0_DQS0N_A)
- new net DQS0NB: U3.B1 (DDR_CH0_DQS0N_B)
- new net DQS0PA: U3.AN1 (DDR_CH0_DQS0P_A)
- new net DQS0PB: U3.B2 (DDR_CH0_DQS0P_B)
- new net DQS1NA: U3.AV3 (DDR_CH0_DQS1N_A)
- new net DQS1NB: U3.K2 (DDR_CH0_DQS1N_B)
- new net DQS1PA: U3.AV4 (DDR_CH0_DQS1P_A)
- new net DQS1PB: U3.K1 (DDR_CH0_DQS1P_B)
- new net EMCIO: C38.1, C40.1, R11.1, R12.1, R9.1, U3.AB35 (EMMCIO_1V8), U3.AC35 (EMMCIO_1V8), U5.C6 (VCCQ), U5.M4 (VCCQ), U5.N4 (VCCQ), U5.P3 (VCCQ), U5.P5 (VCCQ)
- new net RESETA: U3.AG1 (DDR_CH0_RESET_A), U3.P1 (DDR_CH0_RESET_B), U4.T11 (RESET_n)
- new net RST: R9.2, U3.AD40 (EMMC_RSTN/I2C2_SCL_M2/UART5_RTSN_M1/GPIO2_A3_d)
- new net WCK0NA: U3.AR5 (DDR_CH0_WCK0N_A), U4.E3 (DQS0_c_a)
- new net WCK0NB: U3.C3 (DDR_CH0_WCK0N_B), U4.V3 (DQS0_c_b)
- new net WCK0PA: U3.AR6 (DDR_CH0_WCK0P_A), U4.D3 (DQS0_t_a)
- new net WCK0PB: U3.C4 (DDR_CH0_WCK0P_B), U4.W3 (DQS0_t_b)
- new net WCK1NA: U3.AT3 (DDR_CH0_WCK1N_A), U4.E10 (DQS1_c_a)
- new net WCK1NB: U3.E4 (DDR_CH0_WCK1N_B), U4.V10 (DQS1_c_b)
- new net WCK1PA: U3.AT4 (DDR_CH0_WCK1P_A), U4.D10 (DQS1_t_a)
- new net WCK1PB: U3.E3 (DDR_CH0_WCK1P_B), U4.W10 (DQS1_t_b)
- new net ZQA: U3.AM1 (DDR_CH0_ZQ_A)
- new net ZQB: U3.C1 (DDR_CH0_ZQ_B)
- no-connect marks 0 -> 137
Other:
- note added: "DDR"
- note added: "EMMC"
- note added: "SEPERATE SUPPLIES"
- note removed: "LoRaBUSY"
- note removed: "LoRaMISO"
- note removed: "LoRaMOSI"
- note removed: "LoRaNSS"
- note removed: "LoRaRST"
- note removed: "LoRaRX"
- note removed: "LoRaSCK"
- note removed: "LoRaTX"
- note removed: "MUSCSCL"
- note removed: "MUSCSDA"
- note removed: "SCLACCL"
- note removed: "SDAACCL"
- note removed: "SUPPLY FROM STM32"
- moved on the sheet: C1, C2, R1, R2, U2
