File: stemthortyto/stemthortyto.kicad_pcb (KiCad board)
At the start: 8 copper layers, 88.7 x 29.2 mm, 66 parts, among them IC1 E22-900M22S, J1 Jack-DC, Q1 BCV29, U1 LT1585-3.3, U2 ADXL343, U3 RK3588S, U4 K4UCE3Q4AB-MGCL, U5 FEMDRW032G-88A19

Commit message: Add files via upload
Connections:
- U3 pad P1: RESETA -> RESETB
Routing:
- net Net-(U1-GND): track 25.6 -> 0.00 mm
- net RESETA: track 0.00 -> 18.4 mm
- net DQ6B: track 21.0 -> 16.9 mm
- net LoRaRST: track 70.5 -> 67.0 mm
- net A0A: track 19.3 -> 21.0 mm
- net CS0A: track 20.8 -> 20.0 mm, vias 2 -> 1
- net DQ9B: track 21.2 -> 20.5 mm
- net LoRaMISO: track 55.3 -> 54.6 mm
- net DQ4A: track 21.5 -> 20.9 mm
- net GND: track 60.5 -> 60.7 mm, vias 27 -> 67

Commit message: Add files via upload
Routing:
- net CS0A: track 20.0 -> 23.1 mm, vias 1 -> 2
- net A0A: track 21.0 -> 21.9 mm
